File: pcb/kicad/MakersXmasTree_Base/Arbolito.kicad_pcb (KiCad board)
At the start: 2 copper layers, 73 x 66 mm, 58 parts, among them J1 Battery, J2 Header 1x06 2.54mm, P1 USB_C_Plug_USB2.0, Q1 S8050, Q2 S8050, SW1 SW_DPDT_x2, SW2 SW_Push, SW3 SW_Push, SW4 SW_Push, U1 NCP115AMX120TCG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

Commit message: Change R20 with 1K resistor
Parts:
- R20: value 1K8 -> 1K
Changed lines of the file:
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@@
       (effects (font (size 1 1) (thickness 0.15)))
     )
-    (fp_text value "1K8" (at 0 1.65 90) (layer "F.Fab")
+    (fp_text value "1K" (at 0 1.65 90) (layer "F.Fab")
       (effects (font (size 1 1) (thickness 0.15)))
     )
