File: pcb/kicad/Tronco 1 - 8 Leds/Arbolito Tronco.kicad_sch (KiCad schematic)
At the start: 14 parts, among them U1 WS2812B, U2 WS2812B, U3 WS2812B, U4 WS2812B, U5 WS2812B, U6 WS2812B, U7 WS2812B, U8 WS2812B

Commit message: Footprints corrected
Parts:
- added J1, J2, J3, J4, J5, J6: Conn_01x01, Library:Input, symbol Connector_Generic:Conn_01x01
- added J10, J11, J12, J7, J8, J9: Conn_01x01, Library:Output, symbol Connector_Generic:Conn_01x01
Connections:
- net +5V: now also J10.1 (Pin_1), J3.1 (Pin_1), J4.1 (Pin_1), J9.1 (Pin_1)
- net DIN: now also J1.1 (Pin_1), J2.1 (Pin_1)
- net Dout: now also J7.1 (Pin_1), J8.1 (Pin_1)
- net GND: now also J11.1 (Pin_1), J12.1 (Pin_1), J5.1 (Pin_1), J6.1 (Pin_1)

Commit message: Pre USB change
Parts:
- U1, U2, U3, U4, U5, U6, U7, U8: footprint LED_SMD:LED_WS2812B_PLCC4_5.0x5.0mm_P3.2mm -> Library:LED_WS2812B_PLCC4_5.0x5.0mm_P3.2mm
Changed lines of the file:
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@@
       (effects (font (size 1.27 1.27)))
     )
-    (property "Footprint" "LED_SMD:LED_WS2812B_PLCC4_5.0x5.0mm_P3.2mm" (at 270.51 85.09 0)
+    (property "Footprint" "Library:LED_WS2812B_PLCC4_5.0x5.0mm_P3.2mm" (at 270.51 85.09 0)
       (effects (font (size 1.27 1.27)) hide)
     )
@@
       (effects (font (size 1.27 1.27)))
     )
-    (property "Footprint" "LED_SMD:LED_WS2812B_PLCC4_5.0x5.0mm_P3.2mm" (at 182.88 85.09 0)
+    (property "Footprint" "Library:LED_WS2812B_PLCC4_5.0x5.0mm_P3.2mm" (at 182.88 85.09 0)
       (effects (font (size 1.27 1.27)) hide)
     )
@@
       (effects (font (size 1.27 1.27)))
     )
-    (property "Footprint" "LED_SMD:LED_WS2812B_PLCC4_5.0x5.0mm_P3.2mm" (at 29.21 85.09 0)
+    (property "Footprint" "Library:LED_WS2812B_PLCC4_5.0x5.0mm_P3.2mm" (at 29.21 85.09 0)
       (effects (font (size 1.27 1.27)) hide)
     )
@@
       (effects (font (size 1.27 1.27)))
     )
-    (property "Footprint" "LED_SMD:LED_WS2812B_PLCC4_5.0x5.0mm_P3.2mm" (at 110.49 85.09 0)
+    (property "Footprint" "Library:LED_WS2812B_PLCC4_5.0x5.0mm_P3.2mm" (at 110.49 85.09 0)
       (effects (font (size 1.27 1.27)) hide)
     )
@@
       (effects (font (size 1.27 1.27)))
     )
-    (property "Footprint" "LED_SMD:LED_WS2812B_PLCC4_5.0x5.0mm_P3.2mm" (at 48.26 85.09 0)
+    (property "Footprint" "Library:LED_WS2812B_PLCC4_5.0x5.0mm_P3.2mm" (at 48.26 85.09 0)
       (effects (font (size 1.27 1.27)) hide)
     )
@@
       (effects (font (size 1.27 1.27)))
     )
-    (property "Footprint" "LED_SMD:LED_WS2812B_PLCC4_5.0x5.0mm_P3.2mm" (at 158.75 85.09 0)
+    (property "Footprint" "Library:LED_WS2812B_PLCC4_5.0x5.0mm_P3.2mm" (at 158.75 85.09 0)
       (effects (font (size 1.27 1.27)) hide)
     )
@@
       (effects (font (size 1.27 1.27)))
     )
-    (property "Footprint" "LED_SMD:LED_WS2812B_PLCC4_5.0x5.0mm_P3.2mm" (at 134.62 85.09 0)
+    (property "Footprint" "Library:LED_WS2812B_PLCC4_5.0x5.0mm_P3.2mm" (at 134.62 85.09 0)
       (effects (font (size 1.27 1.27)) hide)
     )
@@
       (effects (font (size 1.27 1.27)))
     )
-    (property "Footprint" "LED_SMD:LED_WS2812B_PLCC4_5.0x5.0mm_P3.2mm" (at 250.19 85.09 0)
-      (effects (font (size 1.27 1.27)) hide)
-    )
+    (property "Footprint" "Library:LED_WS2812B_PLCC4_5.0x5.0mm_P3.2mm" (at 250.19 85.09 0)
+      (effects (font (size 1.27 1.27)) hide)
+    )
