File: pcb/kicad/Tronco 2 - 4 Leds/Arbolito Tronco 2.kicad_sch (KiCad schematic)
At the start: 8 parts, among them U1 WS2812B, U2 WS2812B, U3 WS2812B, U4 WS2812B

Commit message: Footprints corrected
Parts:
- added J1, J2, J3, J4, J5, J6: Conn_01x01, Library:Output, symbol Connector_Generic:Conn_01x01
Connections:
- net +5V: now also J3.1 (Pin_1), J4.1 (Pin_1)
- net DIN: now also J1.1 (Pin_1), J2.1 (Pin_1)
- net GND: now also J5.1 (Pin_1), J6.1 (Pin_1)
Changed lines of the file:
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@@
   (junction (at 128.27 127) (diameter 0) (color 0 0 0 0)
   )
+  (junction (at 41.91 111.76) (diameter 0) (color 0 0 0 0)
+  )
   (junction (at 123.19 127) (diameter 0) (color 0 0 0 0)
   )
+  (junction (at 41.91 127) (diameter 0) (color 0 0 0 0)
+  )
   (junction (at 100.33 111.76) (diameter 0) (color 0 0 0 0)
   )
   (junction (at 123.19 111.76) (diameter 0) (color 0 0 0 0)
+  )
+  (junction (at 41.91 143.51) (diameter 0) (color 0 0 0 0)
   )
   (junction (at 100.33 127) (diameter 0) (color 0 0 0 0)
@@
     (stroke (width 0) (type default))
   )
+  (wire (pts (xy 38.1 110.49) (xy 41.91 110.49))
+    (stroke (width 0) (type default))
+  )
   (wire (pts (xy 77.47 111.76) (xy 77.47 115.57))
     (stroke (width 0) (type default))
@@
     (stroke (width 0) (type default))
   )
+  (wire (pts (xy 41.91 143.51) (xy 41.91 146.05))
+    (stroke (width 0) (type default))
+  )
   (wire (pts (xy 128.27 109.22) (xy 128.27 111.76))
     (stroke (width 0) (type default))
   )
   (wire (pts (xy 134.62 111.76) (xy 134.62 115.57))
-    (stroke (width 0) (type default))
-  )
-  (wire (pts (xy 38.1 80.01) (xy 38.1 81.28))
     (stroke (width 0) (type default))
   )
@@
     (stroke (width 0) (type default))
   )
+  (wire (pts (xy 41.91 139.7) (xy 41.91 143.51))
+    (stroke (width 0) (type default))
+  )
   (polyline (pts (xy 31.75 99.06) (xy 271.78 99.06))
     (stroke (width 0.5) (type solid) (color 255 227 36 1))
   )
+  (wire (pts (xy 41.91 110.49) (xy 41.91 111.76))
+    (stroke (width 0) (type default))
+  )
   (polyline (pts (xy 31.75 69.85) (xy 31.75 99.06))
     (stroke (width 0.5) (type solid) (color 255 227 36 1))
@@
     (stroke (width 0) (type default))
   )
+  (wire (pts (xy 41.91 127) (xy 41.91 130.81))
+    (stroke (width 0) (type default))
+  )
   (wire (pts (xy 232.41 80.01) (xy 232.41 81.28))
     (stroke (width 0) (type default))
@@
     (stroke (width 0) (type default))
   )
+  (wire (pts (xy 41.91 125.73) (xy 41.91 127))
+    (stroke (width 0) (type default))
+  )
+  (wire (pts (xy 41.91 111.76) (xy 41.91 115.57))
+    (stroke (width 0) (type default))
+  )
   (wire (pts (xy 123.19 127) (xy 128.27 127))
     (stroke (width 0) (type default))
@@
   (wire (pts (xy 109.22 80.01) (xy 109.22 81.28))
     (stroke (width 0) (type default))
+  )
+  (label "DIN" (at 38.1 110.49 0) (fields_autoplaced)
+    (effects (font (size 1.27 1.27)) (justify left bottom))
   )
   (label "DIN" (at 33.02 85.09 0) (fields_autoplaced)
@@
         (path "/b25a3f48-89a6-49ff-b959-7dc4c52bd0bc"
           (reference "#PWR09") (unit 1)
+        )
+      )
+    )
+  )
+  (symbol (lib_id "Connector_Generic:Conn_01x01") (at 46.99 115.57 0) (unit 1)
+    (in_bom yes) (on_board yes) (dnp no) (fields_autoplaced)
+    (property "Reference" "J2" (at 49.53 114.2999 0)
+      (effects (font (size 1.27 1.27)) (justify left))
+    )
+    (property "Value" "Conn_01x01" (at 49.53 116.8399 0)
+      (effects (font (size 1.27 1.27)) (justify left))
+    )
+    (property "Footprint" "Library:Output" (at 46.99 115.57 0)
+      (effects (font (size 1.27 1.27)) hide)
+    )
+    (property "Datasheet" "~" (at 46.99 115.57 0)
+      (effects (font (size 1.27 1.27)) hide)
+    )
+    (pin "1")
+    (instances
+      (project "Arbolito Tronco 2"
+        (path "/b25a3f48-89a6-49ff-b959-7dc4c52bd0bc"
+          (reference "J2") (unit 1)
+        )
+      )
+    )
+  )
+  (symbol (lib_id "Connector_Generic:Conn_01x01") (at 46.99 111.76 0) (unit 1)
+    (in_bom yes) (on_board yes) (dnp no) (fields_autoplaced)
+    (property "Reference" "J1" (at 49.53 110.4899 0)
+      (effects (font (size 1.27 1.27)) (justify left))
+    )
+    (property "Value" "Conn_01x01" (at 49.53 113.0299 0)
+      (effects (font (size 1.27 1.27)) (justify left))
+    )
+    (property "Footprint" "Library:Output" (at 46.99 111.76 0)
+      (effects (font (size 1.27 1.27)) hide)
+    )
+    (property "Datasheet" "~" (at 46.99 111.76 0)
+      (effects (font (size 1.27 1.27)) hide)
+    )
+    (pin "1")
+    (instances
+      (project "Arbolito Tronco 2"
+        (path "/b25a3f48-89a6-49ff-b959-7dc4c52bd0bc"
+          (reference "J1") (unit 1)
+        )
+      )
+    )
+  )
+  (symbol (lib_id "Connector_Generic:Conn_01x01") (at 46.99 130.81 0) (unit 1)
+    (in_bom yes) (on_board yes) (dnp no) (fields_autoplaced)
+    (property "Reference" "J4" (at 49.53 129.5399 0)
+      (effects (font (size 1.27 1.27)) (justify left))
+    )
+    (property "Value" "Conn_01x01" (at 49.53 132.0799 0)
+      (effects (font (size 1.27 1.27)) (justify left))
+    )
+    (property "Footprint" "Library:Output" (at 46.99 130.81 0)
+      (effects (font (size 1.27 1.27)) hide)
+    )
+    (property "Datasheet" "~" (at 46.99 130.81 0)
+      (effects (font (size 1.27 1.27)) hide)
+    )
+    (pin "1")
+    (instances
+      (project "Arbolito Tronco 2"
+        (path "/b25a3f48-89a6-49ff-b959-7dc4c52bd0bc"
+          (reference "J4") (unit 1)
         )
       )
@@
     )
   )
+  (symbol (lib_id "Connector_Generic:Conn_01x01") (at 46.99 143.51 0) (unit 1)
+    (in_bom yes) (on_board yes) (dnp no) (fields_autoplaced)
+    (property "Reference" "J6" (at 49.53 142.2399 0)
+      (effects (font (size 1.27 1.27)) (justify left))
+    )
+    (property "Value" "Conn_01x01" (at 49.53 144.7799 0)
+      (effects (font (size 1.27 1.27)) (justify left))
+    )
+    (property "Footprint" "Library:Output" (at 46.99 143.51 0)
+      (effects (font (size 1.27 1.27)) hide)
+    )
+    (property "Datasheet" "~" (at 46.99 143.51 0)
+      (effects (font (size 1.27 1.27)) hide)
+    )
+    (pin "1")
+    (instances
+      (project "Arbolito Tronco 2"
+        (path "/b25a3f48-89a6-49ff-b959-7dc4c52bd0bc"
+          (reference "J6") (unit 1)
+        )
+      )
+    )
+  )
   (symbol (lib_id "WB2182:WS2812B") (at 265.43 85.09 0) (unit 1)
     (in_bom yes) (on_board yes) (dnp no) (fields_autoplaced)
@@
     )
   )
+  (symbol (lib_id "Connector_Generic:Conn_01x01") (at 46.99 139.7 0) (unit 1)
+    (in_bom yes) (on_board yes) (dnp no) (fields_autoplaced)
+    (property "Reference" "J5" (at 49.53 138.4299 0)
+      (effects (font (size 1.27 1.27)) (justify left))
+    )
+    (property "Value" "Conn_01x01" (at 49.53 140.9699 0)
+      (effects (font (size 1.27 1.27)) (justify left))
+    )
+    (property "Footprint" "Library:Output" (at 46.99 139.7 0)
+      (effects (font (size 1.27 1.27)) hide)
+    )
+    (property "Datasheet" "~" (at 46.99 139.7 0)
+      (effects (font (size 1.27 1.27)) hide)
+    )
+    (pin "1")
+    (instances
+      (project "Arbolito Tronco 2"
+        (path "/b25a3f48-89a6-49ff-b959-7dc4c52bd0bc"
+          (reference "J5") (unit 1)
+        )
+      )
+    )
+  )
   (symbol (lib_id "power:+5V") (at 109.22 80.01 0) (unit 1)
     (in_bom yes) (on_board yes) (dnp no) (fields_autoplaced)
@@
     )
   )
+  (symbol (lib_id "power:GND") (at 41.91 146.05 0) (unit 1)
+    (in_bom yes) (on_board yes) (dnp no)
+    (property "Reference" "#PWR012" (at 41.91 152.4 0)
+      (effects (font (size 1.27 1.27)) hide)
+    )
+    (property "Value" "GND" (at 41.91 149.86 0)
+      (effects (font (size 1.27 1.27)))
+    )
+    (property "Footprint" "" (at 41.91 146.05 0)
+      (effects (font (size 1.27 1.27)) hide)
+    )
+    (property "Datasheet" "" (at 41.91 146.05 0)
+      (effects (font (size 1.27 1.27)) hide)
+    )
+    (pin "1")
+    (instances
+      (project "Arbolito Tronco 2"
+        (path "/b25a3f48-89a6-49ff-b959-7dc4c52bd0bc"
+          (reference "#PWR012") (unit 1)
+        )
+      )
+    )
+  )
   (symbol (lib_id "WB2182:WS2812B") (at 118.11 85.09 0) (unit 1)
     (in_bom yes) (on_board yes) (dnp no) (fields_autoplaced)
@@
     )
   )
+  (symbol (lib_id "power:+5V") (at 41.91 125.73 0) (unit 1)
+    (in_bom yes) (on_board yes) (dnp no)
+    (property "Reference" "#PWR011" (at 41.91 129.54 0)
+      (effects (font (size 1.27 1.27)) hide)
+    )
+    (property "Value" "+5V" (at 41.91 120.65 0)
+      (effects (font (size 1.27 1.27)))
+    )
+    (property "Footprint" "" (at 41.91 125.73 0)
+      (effects (font (size 1.27 1.27)) hide)
+    )
+    (property "Datasheet" "" (at 41.91 125.73 0)
+      (effects (font (size 1.27 1.27)) hide)
+    )
+    (pin "1")
+    (instances
+      (project "Arbolito Tronco 2"
+        (path "/b25a3f48-89a6-49ff-b959-7dc4c52bd0bc"
+          (reference "#PWR011") (unit 1)
+        )
+      )
+    )
+  )
   (symbol (lib_id "power:GND") (at 85.09 90.17 0) (unit 1)
     (in_bom yes) (on_board yes) (dnp no) (fields_autoplaced)
@@
         )
       )
+    )
+  )
+  (symbol (lib_id "Connector_Generic:Conn_01x01") (at 46.99 127 0) (unit 1)
+    (in_bom yes) (on_board yes) (dnp no) (fields_autoplaced)
+    (property "Reference" "J3" (at 49.53 125.7299 0)
+      (effects (font (size 1.27 1.27)) (justify left))
+    )
+    (property "Value" "Conn_01x01" (at 49.53 128.2699 0)
+      (effects (font (size 1.27 1.27)) (justify left))
+    )
+    (property "Footprint" "Library:Output" (at 46.99 127 0)
+      (effects (font (size 1.27 1.27)) hide)
+    )
+    (property "Datasheet" "~" (at 46.99 127 0)
+      (effects (font (size 1.27 1.27)) hide)
+    )
+    (pin "1")
+    (instances
+      (project "Arbolito Tronco 2"
+        (path "/b25a3f48-89a6-49ff-b959-7dc4c52bd0bc"
+          (reference "J3") (unit 1)
+        )
+      )

Commit message: Led Footprint Changed
Parts:
- U1, U2, U3, U4: footprint LED_SMD:LED_WS2812B_PLCC4_5.0x5.0mm_P3.2mm -> Library:LED_WS2812B_PLCC4_5.0x5.0mm_P3.2mm
Changed lines of the file:
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@@
       (effects (font (size 1.27 1.27)))
     )
-    (property "Footprint" "LED_SMD:LED_WS2812B_PLCC4_5.0x5.0mm_P3.2mm" (at 93.98 85.09 0)
+    (property "Footprint" "Library:LED_WS2812B_PLCC4_5.0x5.0mm_P3.2mm" (at 93.98 85.09 0)
       (effects (font (size 1.27 1.27)) hide)
     )
@@
       (effects (font (size 1.27 1.27)))
     )
-    (property "Footprint" "LED_SMD:LED_WS2812B_PLCC4_5.0x5.0mm_P3.2mm" (at 265.43 85.09 0)
+    (property "Footprint" "Library:LED_WS2812B_PLCC4_5.0x5.0mm_P3.2mm" (at 265.43 85.09 0)
       (effects (font (size 1.27 1.27)) hide)
     )
@@
       (effects (font (size 1.27 1.27)))
     )
-    (property "Footprint" "LED_SMD:LED_WS2812B_PLCC4_5.0x5.0mm_P3.2mm" (at 241.3 85.09 0)
+    (property "Footprint" "Library:LED_WS2812B_PLCC4_5.0x5.0mm_P3.2mm" (at 241.3 85.09 0)
       (effects (font (size 1.27 1.27)) hide)
     )
@@
       (effects (font (size 1.27 1.27)))
     )
-    (property "Footprint" "LED_SMD:LED_WS2812B_PLCC4_5.0x5.0mm_P3.2mm" (at 118.11 85.09 0)
-      (effects (font (size 1.27 1.27)) hide)
-    )
+    (property "Footprint" "Library:LED_WS2812B_PLCC4_5.0x5.0mm_P3.2mm" (at 118.11 85.09 0)
+      (effects (font (size 1.27 1.27)) hide)
+    )
