File: pcb/kicad/Tronco 2/Arbolito Tronco 2.kicad_pcb (KiCad board)
At the start: 2 copper layers, 68.2 x 111 mm, 34 parts, among them U1 WS2812B, U10 WS2812B, U11 WS2812B, U12 WS2812B, U2 WS2812B, U3 WS2812B, U4 WS2812B, U5 WS2812B, U6 WS2812B, U7 WS2812B, U8 WS2812B, U9 WS2812B

Commit message: Do some cleaning and add .gitignore
Parts:
- removed C3, C4: 0.1uF, Capacitor_SMD:C_0805_2012Metric
- removed the U1 at (117.1, 110.0)
- removed U11, U12, U5, U6, U7, U8: WS2812B, LED_SMD:LED_WS2812B_PLCC4_5.0x5.0mm_P3.2mm
- removed the U2 at (117.1, 110.0)
- added J1: Conn_01x01, Library:Output, F.Cu at (138.3, 65.1)
- added J2: Conn_01x01, Library:Output, F.Cu at (140.7, 65.1)
- added J3: Conn_01x01, Library:Output, F.Cu at (138.3, 62.1)
- added J4: Conn_01x01, Library:Output, F.Cu at (140.7, 62.1)
- added J5: Conn_01x01, Library:Output, F.Cu at (140.7, 68.1)
- added J6: Conn_01x01, Library:Output, F.Cu at (138.3, 68.1)
- U1: renamed from U3; footprint LED_SMD:LED_WS2812B_PLCC4_5.0x5.0mm_P3.2mm -> Library:LED_WS2812B_PLCC4_5.0x5.0mm_P3.2mm
- U2: renamed from U4; footprint LED_SMD:LED_WS2812B_PLCC4_5.0x5.0mm_P3.2mm -> Library:LED_WS2812B_PLCC4_5.0x5.0mm_P3.2mm
- U3: renamed from U9; footprint LED_SMD:LED_WS2812B_PLCC4_5.0x5.0mm_P3.2mm -> Library:LED_WS2812B_PLCC4_5.0x5.0mm_P3.2mm
- U4: renamed from U10; footprint LED_SMD:LED_WS2812B_PLCC4_5.0x5.0mm_P3.2mm -> Library:LED_WS2812B_PLCC4_5.0x5.0mm_P3.2mm
- moved C2 31.7 mm to (148.8, 81.2)
- moved C5 31.7 mm to (148.8, 81.2)
Connections:
- U1 pad 4: Net-(U2-DOUT) -> /DIN
- U2 pad 2: Net-(U4-DOUT) -> Net-(U2-DOUT)
- U3 pad 4: Net-(U8-DOUT) -> Net-(U2-DOUT)
- U4 pad 2: Net-(U10-DOUT) -> unconnected-(U4-DOUT-Pad2)
Routing:
- net Net-(U10-DOUT): track 39.9 -> 0.00 mm
- net Net-(U4-DOUT): track 38.1 -> 0.00 mm
- net Net-(U8-DOUT): track 35.3 -> 0.00 mm
- net /DIN: track 55.7 -> 29.0 mm
- net Net-(U6-DOUT): track 21.5 -> 0.00 mm
- net +5V: track 26.8 -> 14.8 mm, vias 10 -> 6
- net GND: track 26.4 -> 14.4 mm, vias 10 -> 6
- net Net-(U2-DOUT): track 49.4 -> 39.7 mm
- net Net-(U1-DOUT) (its old number): track 3.54 -> 0.00 mm, vias 1 -> 0
- net Net-(U5-DOUT): track 3.35 -> 0.00 mm, vias 1 -> 0
- net Net-(U7-DOUT): track 3.35 -> 0.00 mm, vias 1 -> 0
- net Net-(U11-DOUT): track 3.35 -> 0.00 mm, vias 1 -> 0
- removed copper zone on B.Cu, net +5V
- removed copper zone on B.Cu, net /DIN
- removed copper zone on F.Cu, net /DIN
- removed copper zone on F.Cu, net GND
Other:
- outline, holes or cut-outs redrawn
