File: pcb/kicad/Tronco 2/Arbolito Tronco 2.kicad_pcb (KiCad board)
At the start: 2 copper layers, 68.2 x 111 mm, 30 parts, among them J1 Conn_01x01, J2 Conn_01x01, J3 Conn_01x01, J4 Conn_01x01, J5 Conn_01x01, J6 Conn_01x01, U1 WS2812B, U2 WS2812B, U3 WS2812B, U4 WS2812B

Commit message: Led Shorts fixed
Vias were shorting leds pins, should be fixed :)
Routing:
- net Net-(U2-DOUT): track 39.7 -> 43.1 mm

Commit message: DRC Errors fixeds
The WS218B double footprint was remade in order to avoid DRC errors :3
Parts:
- added J10: Conn_01x01, Library:Output, B.Cu at (140.7, 62.1)
- added J11: Conn_01x01, Library:Output, B.Cu at (140.8, 68.1)
- added J12: Conn_01x01, Library:Output, B.Cu at (138.3, 68.1)
- added J7: Conn_01x01, Library:Output, B.Cu at (140.7, 65.1)
- added J8: Conn_01x01, Library:Output, B.Cu at (138.3, 65.1)
- added J9: Conn_01x01, Library:Output, B.Cu at (138.3, 62.1)
